File: Schematic & Board/LEDStatusBoard.brd (EAGLE design)
At the start: 53.3 x 92.4 mm, 35 parts, among them J1 0768250002, U1 MIC5219-5.0YM5-TR, U2 74HCT4053D, U3 74HCT4053D, U4 74HCT4053D

Commit message: Clean up repository
Parts:
- removed 470PF: CGA1A2X7R1H471K030BA, CGA1A2X7R1H471K030BA:CAP_0603_TDK
- added C2: 1206AA471JAT1A, 1206AA471JAT1A:CAP_1206_AVX
Connections:
- net GND: now also C2.1; no longer 470PF.1
- net N$1: now also C2.2; no longer 470PF.2
Routing:
- net N$1: track 2.09 -> 15.7 mm
Other:
- board size 53.3 x 92.4 mm -> 53.3 x 94.4 mm
- board text added: "12V"
- board text added: "12V Step-Down"
- board text added: "2.2 uF Output Capacitor"
- board text added: "470 pF Bypass Capacitor"
- board text added: "74HCT4053D"
- board text added: "91 Ω"
- board text added: "Arm"
- board text added: "Back Camera"
- board text added: "Cam 1"
- board text added: "Cam 2"
- board text added: "Cam 3"
- board text added: "Controls System Status Board Board Created By: Moustafa Eid Date Created: 10-19-2020"
- board text added: "Drive"
- board text added: "Enc"
- board text added: "Encoders"
- board text added: "Front Camera"
- board text added: "GND"
- board text added: "Jetson Nano"
- board text added: "MIC5219-5-0YM5-TR 12V to 5V LDO"
- board text added: "Nano"
- board text added: "Power Input"
- board text added: "Third Camera"
- board text added: "Vin"
