File: Schematic & Board/LEDStatusBoard.sch (EAGLE design)
At the start: 35 parts, among them J1 0768250002, U1 MIC5219-5.0YM5-TR, U2 74HCT4053D, U3 74HCT4053D, U4 74HCT4053D

Commit message: Clean up repository
Parts:
- removed 470PF: CGA1A2X7R1H471K030BA, CGA1A2X7R1H471K030BA:CGA1A2X7R1H471K030BA
- added C2: 1206AA471JAT1A, 1206AA471JAT1A:1206AA471JAT1A
Connections:
- net GND: now also C2.1; no longer 470PF.1
- net N$1: now also C2.2; no longer 470PF.2
- net R1: no longer U4.1Y0
- net R7: now also U4.1Y0
